File: hardware/at2usb/at2usb.kicad_pcb (KiCad board)
At the start: 2 copper layers, 46.5 x 25.5 mm, 8 parts, among them J1 AT (PS/2) keyboard, J2 UART, J3 USB connector breakout board, J4 Programmer, U1 PIC16F1459-IP

Commit message: Add gnd pin next to uart pins
Parts:
- J2: footprint Connector_PinHeader_2.54mm:PinHeader_1x02_P2.54mm_Vertical -> Connector_PinHeader_2.54mm:PinHeader_1x03_P2.54mm_Vertical
- moved J2 1.57 mm to (142.5, 52.5)
Changed lines of the file:
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@@
     )
   )
-  (footprint "Connector_PinHeader_2.54mm:PinHeader_1x02_P2.54mm_Vertical" (layer "F.Cu")
-    (at 142.89 54)
-    (descr "Through hole straight pin header, 1x02, 2.54mm pitch, single row")
-    (tags "Through hole pin header THT 1x02 2.54mm single row")
+  (footprint "Connector_PinHeader_2.54mm:PinHeader_1x03_P2.54mm_Vertical" (layer "F.Cu")
+    (at 142.5 52.475)
+    (descr "Through hole straight pin header, 1x03, 2.54mm pitch, single row")
+    (tags "Through hole pin header THT 1x03 2.54mm single row")
     (property "Sheetfile" "at2usb.kicad_sch")
     (property "Sheetname" "")
-    (property "ki_description" "Generic connector, single row, 01x02, script generated")
+    (property "ki_description" "Generic connector, single row, 01x03, script generated")
     (property "ki_keywords" "connector")
     (attr through_hole)
@@
         (effects (font (size 1 1) (thickness 0.15)))
     )
-    (fp_text value "UART" (at 0 4.87) (layer "F.Fab")
-        (effects (font (size 1 1) (thickness 0.15)))
-    )
-    (fp_text user "${REFERENCE}" (at 0 1.27 90) (layer "F.Fab")
+    (fp_text value "UART" (at 0 7.41) (layer "F.Fab")
+        (effects (font (size 1 1) (thickness 0.15)))
+    )
+    (fp_text user "${REFERENCE}" (at 0 2.54 90) (layer "F.Fab")
         (effects (font (size 1 1) (thickness 0.15)))
     )
@@
     (fp_line (start -1.33 0) (end -1.33 -1.33)
       (stroke (width 0.12) (type solid)) (layer "F.SilkS"))
-    (fp_line (start -1.33 1.27) (end -1.33 3.87)
+    (fp_line (start -1.33 1.27) (end -1.33 6.41)
       (stroke (width 0.12) (type solid)) (layer "F.SilkS"))
     (fp_line (start -1.33 1.27) (end 1.33 1.27)
       (stroke (width 0.12) (type solid)) (layer "F.SilkS"))
-    (fp_line (start -1.33 3.87) (end 1.33 3.87)
-      (stroke (width 0.12) (type solid)) (layer "F.SilkS"))
-    (fp_line (start 1.33 1.27) (end 1.33 3.87)
-      (stroke (width 0.12) (type solid)) (layer "F.SilkS"))
-    (fp_line (start -1.8 -1.8) (end -1.8 4.35)
-      (stroke (width 0.05) (type solid)) (layer "F.CrtYd"))
-    (fp_line (start -1.8 4.35) (end 1.8 4.35)
+    (fp_line (start -1.33 6.41) (end 1.33 6.41)
+      (stroke (width 0.12) (type solid)) (layer "F.SilkS"))
+    (fp_line (start 1.33 1.27) (end 1.33 6.41)
+      (stroke (width 0.12) (type solid)) (layer "F.SilkS"))
+    (fp_line (start -1.8 -1.8) (end -1.8 6.85)
+      (stroke (width 0.05) (type solid)) (layer "F.CrtYd"))
+    (fp_line (start -1.8 6.85) (end 1.8 6.85)
       (stroke (width 0.05) (type solid)) (layer "F.CrtYd"))
     (fp_line (start 1.8 -1.8) (end -1.8 -1.8)
       (stroke (width 0.05) (type solid)) (layer "F.CrtYd"))
-    (fp_line (start 1.8 4.35) (end 1.8 -1.8)
+    (fp_line (start 1.8 6.85) (end 1.8 -1.8)
       (stroke (width 0.05) (type solid)) (layer "F.CrtYd"))
     (fp_line (start -1.27 -0.635) (end -0.635 -1.27)
       (stroke (width 0.1) (type solid)) (layer "F.Fab"))
-    (fp_line (start -1.27 3.81) (end -1.27 -0.635)
+    (fp_line (start -1.27 6.35) (end -1.27 -0.635)
       (stroke (width 0.1) (type solid)) (layer "F.Fab"))
     (fp_line (start -0.635 -1.27) (end 1.27 -1.27)
       (stroke (width 0.1) (type solid)) (layer "F.Fab"))
-    (fp_line (start 1.27 -1.27) (end 1.27 3.81)
-      (stroke (width 0.1) (type solid)) (layer "F.Fab"))
-    (fp_line (start 1.27 3.81) (end -1.27 3.81)
+    (fp_line (start 1.27 -1.27) (end 1.27 6.35)
+      (stroke (width 0.1) (type solid)) (layer "F.Fab"))
+    (fp_line (start 1.27 6.35) (end -1.27 6.35)
       (stroke (width 0.1) (type solid)) (layer "F.Fab"))
     (pad "1" thru_hole rect (at 0 0) (size 1.7 1.7) (drill 1) (layers "*.Cu" "*.Mask")
@@
     (pad "2" thru_hole oval (at 0 2.54) (size 1.7 1.7) (drill 1) (layers "*.Cu" "*.Mask")
       (net 7 "/UART_TX") (pinfunction "Pin_2") (pintype "passive"))
-    (model "${KICAD6_3DMODEL_DIR}/Connector_PinHeader_2.54mm.3dshapes/PinHeader_1x02_P2.54mm_Vertical.wrl"
+    (pad "3" thru_hole oval (at 0 5.08) (size 1.7 1.7) (drill 1) (layers "*.Cu" "*.Mask")
+      (net 2 "GND") (pinfunction "Pin_3") (pintype "passive"))
+    (model "${KICAD6_3DMODEL_DIR}/Connector_PinHeader_2.54mm.3dshapes/PinHeader_1x03_P2.54mm_Vertical.wrl"
       (offset (xyz 0 0 0))
       (scale (xyz 1 1 1))
@@
   (segment (start 117.65 59.76) (end 117.65 58.62) (width 1) (layer "B.Cu") (net 5))
   (segment (start 120.15 63) (end 120.15 62.26) (width 1) (layer "B.Cu") (net 5))
-  (segment (start 138.43 54) (end 142.89 54) (width 1) (layer "B.Cu") (net 6))
-  (segment (start 135.43 51) (end 138.43 54) (width 1) (layer "B.Cu") (net 6))
-  (segment (start 140.05 56.54) (end 142.89 56.54) (width 1) (layer "B.Cu") (net 7))
-  (segment (start 140.05 56.54) (end 137.97 58.62) (width 1) (layer "B.Cu") (net 7))
+  (segment (start 136 53) (end 141.975 53) (width 1) (layer "B.Cu") (net 6))
+  (segment (start 135.43 52.43) (end 136 53) (width 1) (layer "B.Cu") (net 6))
+  (segment (start 135.43 51) (end 135.43 52.43) (width 1) (layer "B.Cu") (net 6))
+  (segment (start 141.975 53) (end 142.5 52.475) (width 1) (layer "B.Cu") (net 6))
+  (segment (start 141.575 55.015) (end 137.97 58.62) (width 1) (layer "B.Cu") (net 7))
+  (segment (start 142.5 55.015) (end 141.575 55.015) (width 1) (layer "B.Cu") (net 7))
   (segment (start 125.61 61.5) (end 122.73 58.62) (width 1) (layer "B.Cu") (net 8))
   (segment (start 144.39 61.5) (end 125.61 61.5) (width 1) (layer "B.Cu") (net 8))

Commit message: Add MCLR pull-up resistor in schematic, remove UART RX
Parts:
- added R1: 10k, Resistor_THT:R_Axial_DIN0207_L6.3mm_D2.5mm_P2.54mm_Vertical, F.Cu at (128.0, 64.0)
Changed lines of the file:
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@@
     (property "ki_keywords" "connector")
     (attr through_hole)
-    (fp_text reference "J2" (at 0 -2.33) (layer "F.SilkS")
+    (fp_text reference "J2" (at -1 -1.975) (layer "F.SilkS")
         (effects (font (size 1 1) (thickness 0.15)))
     )
@@
       (net 2 "GND") (pintype "passive"))
     (model "${KICAD6_3DMODEL_DIR}/Capacitor_THT.3dshapes/CP_Radial_D5.0mm_P2.00mm.wrl"
+      (offset (xyz 0 0 0))
+      (scale (xyz 1 1 1))
+      (rotate (xyz 0 0 0))
+    )
+  )
+  (footprint "Resistor_THT:R_Axial_DIN0207_L6.3mm_D2.5mm_P2.54mm_Vertical" (layer "F.Cu")
+    (at 128 64.045 90)
+    (descr "Resistor, Axial_DIN0207 series, Axial, Vertical, pin pitch=2.54mm, 0.25W = 1/4W, length*diameter=6.3*2.5mm^2, http://cdn-reichelt.de/documents/datenblatt/B400/1_4W%23YAG.pdf")
+    (tags "Resistor Axial_DIN0207 series Axial Vertical pin pitch 2.54mm 0.25W = 1/4W length 6.3mm diameter 2.5mm")
+    (property "Sheetfile" "at2usb.kicad_sch")
+    (property "Sheetname" "")
+    (property "ki_description" "Resistor, US symbol")
+    (property "ki_keywords" "R res resistor")
+    (attr through_hole)
+    (fp_text reference "R1" (at 1 3 180) (layer "F.SilkS")
+        (effects (font (size 1 1) (thickness 0.15)))
+    )
+    (fp_text value "10k" (at 1.27 2.37 90) (layer "F.Fab")
+        (effects (font (size 1 1) (thickness 0.15)))
+    )
+    (fp_text user "${REFERENCE}" (at 1.27 -2.37 90) (layer "F.Fab")
+        (effects (font (size 1 1) (thickness 0.15)))
+    )
+    (fp_line (start 1.37 0) (end 1.44 0)
+      (stroke (width 0.12) (type solid)) (layer "F.SilkS"))
+    (fp_circle (center 0 0) (end 1.37 0)
+      (stroke (width 0.12) (type solid)) (fill none) (layer "F.SilkS"))
+    (fp_line (start -1.5 -1.5) (end -1.5 1.5)
+      (stroke (width 0.05) (type solid)) (layer "F.CrtYd"))
+    (fp_line (start -1.5 1.5) (end 3.59 1.5)
+      (stroke (width 0.05) (type solid)) (layer "F.CrtYd"))
+    (fp_line (start 3.59 -1.5) (end -1.5 -1.5)
+      (stroke (width 0.05) (type solid)) (layer "F.CrtYd"))
+    (fp_line (start 3.59 1.5) (end 3.59 -1.5)
+      (stroke (width 0.05) (type solid)) (layer "F.CrtYd"))
+    (fp_line (start 0 0) (end 2.54 0)
+      (stroke (width 0.1) (type solid)) (layer "F.Fab"))
+    (fp_circle (center 0 0) (end 1.25 0)
+      (stroke (width 0.1) (type solid)) (fill none) (layer "F.Fab"))
+    (pad "1" thru_hole circle (at 0 0 90) (size 1.6 1.6) (drill 0.8) (layers "*.Cu" "*.Mask")
+      (net 3 "+5V") (pintype "passive"))
+    (pad "2" thru_hole oval (at 2.54 0 90) (size 1.6 1.6) (drill 0.8) (layers "*.Cu" "*.Mask")
+      (net 8 "/{slash}MCLR") (pintype "passive"))
+    (model "${KICAD6_3DMODEL_DIR}/Resistor_THT.3dshapes/R_Axial_DIN0207_L6.3mm_D2.5mm_P2.54mm_Vertical.wrl"
       (offset (xyz 0 0 0))
       (scale (xyz 1 1 1))
@@
   (segment (start 113.39 51) (end 111.89 49.5) (width 1) (layer "B.Cu") (net 2))
   (segment (start 115.11 51) (end 113.39 51) (width 1) (layer "B.Cu") (net 2))
-  (segment (start 139.85 43.797919) (end 139.85 45) (width 1) (layer "B.Cu") (net 3))
-  (segment (start 143.94 43.45) (end 140.197919 43.45) (width 1) (layer "B.Cu") (net 3))
-  (segment (start 119.61 65) (end 142.89 65) (width 1) (layer "B.Cu") (net 3))
+  (segment (start 127.045 65) (end 128 64.045) (width 1) (layer "B.Cu") (net 3))
+  (segment (start 143.845 64.045) (end 147.59 60.3) (width 1) (layer "B.Cu") (net 3))
+  (segment (start 140.197919 43.45) (end 139.85 43.797919) (width 1) (layer "B.Cu") (net 3))
+  (segment (start 128 64.045) (end 143.845 64.045) (width 1) (layer "B.Cu") (net 3))
   (segment (start 115.11 59.72) (end 117.61 62.22) (width 1) (layer "B.Cu") (net 3))
   (segment (start 114.73 59) (end 115.11 58.62) (width 1) (layer "B.Cu") (net 3))
   (segment (start 117.61 62.22) (end 117.61 63) (width 1) (layer "B.Cu") (net 3))
+  (segment (start 147.59 60.3) (end 147.59 47.1) (width 1) (layer "B.Cu") (net 3))
   (segment (start 115.11 58.62) (end 115.11 59.72) (width 1) (layer "B.Cu") (net 3))
+  (segment (start 147.59 47.1) (end 143.94 43.45) (width 1) (layer "B.Cu") (net 3))
   (segment (start 115.11 56.464888) (end 115.11 58.62) (width 1) (layer "B.Cu") (net 3))
   (segment (start 108.345112 51.5) (end 108.345112 49.424888) (width 1) (layer "B.Cu") (net 3))
+  (segment (start 139.85 43.797919) (end 139.85 45) (width 1) (layer "B.Cu") (net 3))
   (segment (start 108.345112 49.424888) (end 112.77 45) (width 1) (layer "B.Cu") (net 3))
+  (segment (start 117.61 63) (end 119.61 65) (width 1) (layer "B.Cu") (net 3))
+  (segment (start 119.61 65) (end 127.045 65) (width 1) (layer "B.Cu") (net 3))
   (segment (start 108.345112 51.5) (end 110.145112 51.5) (width 1) (layer "B.Cu") (net 3))
   (segment (start 108.345112 59) (end 114.73 59) (width 1) (layer "B.Cu") (net 3))
   (segment (start 110.145112 51.5) (end 115.11 56.464888) (width 1) (layer "B.Cu") (net 3))
-  (segment (start 147.59 47.1) (end 143.94 43.45) (width 1) (layer "B.Cu") (net 3))
-  (segment (start 119.61 65) (end 117.61 63) (width 1) (layer "B.Cu") (net 3))
-  (segment (start 140.197919 43.45) (end 139.85 43.797919) (width 1) (layer "B.Cu") (net 3))
-  (segment (start 142.89 65) (end 147.59 60.3) (width 1) (layer "B.Cu") (net 3))
-  (segment (start 147.59 60.3) (end 147.59 47.1) (width 1) (layer "B.Cu") (net 3))
+  (segment (start 143.94 43.45) (end 140.197919 43.45) (width 1) (layer "B.Cu") (net 3))
   (segment (start 122.69 62.3) (end 122.69 63) (width 1) (layer "B.Cu") (net 4))
   (segment (start 120.19 58.62) (end 120.19 59.8) (width 1) (layer "B.Cu") (net 4))
@@
   (segment (start 141.575 55.015) (end 137.97 58.62) (width 1) (layer "B.Cu") (net 7))
   (segment (start 142.5 55.015) (end 141.575 55.015) (width 1) (layer "B.Cu") (net 7))
-  (segment (start 125.61 61.5) (end 122.73 58.62) (width 1) (layer "B.Cu") (net 8))
-  (segment (start 144.39 61.5) (end 125.61 61.5) (width 1) (layer "B.Cu") (net 8))
-  (segment (start 142.39 45) (end 146.39 49) (width 1) (layer "B.Cu") (net 8))
-  (segment (start 146.39 59.5) (end 144.39 61.5) (width 1) (layer "B.Cu") (net 8))
-  (segment (start 146.39 49) (end 146.39 59.5) (width 1) (layer "B.Cu") (net 8))
+  (segment (start 122.73 58.62) (end 125.61 61.5) (width 1) (layer "B.Cu") (net 8))
+  (segment (start 142.39 45) (end 146.29 48.9) (width 1.2) (layer "B.Cu") (net 8))
+  (segment (start 146.29 48.9) (end 146.29 49.5) (width 1.2) (layer "B.Cu") (net 8))
+  (segment (start 125.61 61.5) (end 144.39 61.5) (width 1) (layer "B.Cu") (net 8))
+  (segment (start 144.39 61.5) (end 146.39 59.5) (width 1) (layer "B.Cu") (net 8))
+  (segment (start 146.39 59.5) (end 146.39 49.5) (width 1) (layer "B.Cu") (net 8))
   (segment (start 130.39 43) (end 133.89 43) (width 1) (layer "B.Cu") (net 9))
   (segment (start 129.89 46.38) (end 129.89 43.5) (width 1) (layer "B.Cu") (net 9))
